File: mold_detect.kicad_pcb (KiCad board)
At the start: 2 copper layers, 37 x 68 mm, 22 parts, among them J1 ISP, SW1 watchdog_sw, U1 SHT30-DIS, U2 TPL5010, U3 ATmega328P-P

Commit message: added ces reference; moved sensor to bottom
Parts:
- added G***: LOGO, Library:kit_logo, F.Cu at (85.0, 132.5)
- R1, R2, R3, R4, R5, R6: footprint Resistor_SMD:R_0201_0603Metric -> Resistor_SMD:R_0603_1608Metric
- REF**: moved to F.Cu
- moved R6 63.4 mm to (93.1, 145.2)
- moved U1 63.0 mm to (90.5, 143.6)
- moved C1 62.9 mm to (87.8, 143.6)
- moved R5 62.6 mm to (93.1, 142.1)
- moved REF** 15.9 mm to (99.0, 135.0), turned to 90 degrees
- moved R2 6.75 mm to (103.9, 146.5)
- moved Red1 6.21 mm to (100.0, 144.5)
- moved R1 5.11 mm to (100.8, 146.5)
- moved U2 4.32 mm to (92.9, 82.8)
- moved SW1 4.27 mm to (100.3, 82.4)
- moved Blue1 4.25 mm to (104.7, 144.5)
- moved R3 3.89 mm to (90.0, 83.0)
- moved R4 0.88 mm to (106.0, 86.3)
Routing:
- net SCL: track 12.2 -> 68.4 mm, vias 0 -> 2
- net SDA: track 13.4 -> 67.7 mm, vias 0 -> 2
- net +3V0: track 136.9 -> 162.6 mm, vias 0 -> 2
- net DONE: track 21.0 -> 16.5 mm
- net WAKE_INTR: track 20.4 -> 15.8 mm
- net HUM_LED: track 32.9 -> 29.6 mm
- net RST: track 59.4 -> 56.8 mm
- net SCK: track 25.3 -> 23.2 mm
- net MISO: track 18.6 -> 17.0 mm
- net Net-(Red1-K): track 3.55 -> 2.03 mm
- net TEMP_LED: track 27.6 -> 26.2 mm
- net Net-(Blue1-K): track 3.10 -> 2.05 mm
Other:
- board text added: "github.com/christopher-besch/mold_detect Christopher Besch <mail@chris-besch.com> designed at Chair for Embedded Systems Rev. 1.0.0 January 2024"
- board text removed: "github.com/christopher-besch/mold_detect Christopher Besch <mail@chris-besch.com> Rev. 1.0.0 January 2024"
